File: circuit/RLCMeterH750/RLCMeterH750.kicad_pcb (KiCad board)
At the start: 2 copper layers, 80 x 65 mm, 142 parts, among them J1 SWD, J2 USB_B_Micro, J3 ILI_9321(2.2inch), J4 DUT, SW1 EVQWKL001, SW2 PowerOn, U1 STM32H750VITx, U10 AD8031, U11 AD8031, U12 AD9833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

Commit message: - немного причесали внешний вид платы
Parts:
- added BalmerDX: balmer, balmer:balmer_logo, B.Cu at (155.2, 124.6)
- added REF**: Pin_D1.3mm_L10.0mm_W3.5mm_Flat, Connector_Pin:Pin_D1.3mm_L10.0mm_W3.5mm_Flat, F.Cu at (108.0, 133.1)
- moved C3 2.22 mm to (177.8, 101.8)
Routing:
- net /NRST: track 38.4 -> 40.8 mm
- net GND: track 228.7 -> 227.9 mm, vias 162 -> 173
Other:
- board text added: "BalmerDX 2019"
