File: circuit/RLCMeterH750/analog.sch (KiCad schematic (older format))
At the start: 33 parts

Commit message: - вродебы нарисовали аналоговую часть
Parts:
- removed C?: 100n, symbol Device:C
- added C? (x8): 100n, Capacitor_SMD:C_0603_1608Metric, symbol Device:C
- added C? (x2): 330p, Capacitor_SMD:C_1206_3216Metric, symbol Device:C
- added C? (x2): 22n, Capacitor_SMD:C_0603_1608Metric, symbol Device:C
- added C?: 560p, Capacitor_SMD:C_1206_3216Metric, symbol Device:C
- added C? (x2): 180p, Capacitor_SMD:C_1206_3216Metric, symbol Device:C
- added C? (x2): 10u, Capacitor_SMD:C_1206_3216Metric, symbol Device:C
- added J?: DUT, Connector_PinHeader_2.54mm:PinHeader_1x04_P2.54mm_Vertical, symbol Connector_Generic:Conn_01x04
- added R? (x13): 1k, Resistor_SMD:R_0603_1608Metric, symbol Device:R
- added R? (x2): 2k, Resistor_SMD:R_0603_1608Metric, symbol Device:R
- added R?: 360, Resistor_SMD:R_0603_1608Metric, symbol Device:R
- added R?: 510, Resistor_SMD:R_0603_1608Metric, symbol Device:R
- added R?: 12k, Resistor_SMD:R_0603_1608Metric, symbol Device:R
- added R? (x2): 100, Resistor_SMD:R_0603_1608Metric, symbol Device:R
- added R?: 27k, Resistor_SMD:R_0603_1608Metric, symbol Device:R
- added R?: 10k, Resistor_SMD:R_0603_1608Metric, symbol Device:R
- added U? (x3): AD8031, Package_TO_SOT_SMD:SOT-23-5, symbol Amplifier_Operational:MCP6001-OT
- added U?: AD8221BRMZ, Package_SO:MSOP-8_3x3mm_P0.65mm, symbol Amplifier_Instrumentation:AD8421BRMZ
- added U?: FSA3357L8X, balmer:MicroPak_8-Lead, symbol balmer:FSA3357L8X
- C?: value 1.5n -> 560p
- C?: value 25u -> 100u
- R?: value 1k -> 2k
- R?: value 510 -> 360
- R?: value 1k -> 510
- R?: value 5.1k -> 12k
Connections:
- net labels added: ADC12_INP4, S1, S2
- wire segments 68 -> 195
Other:
- note added: "0.2V p-p"
- note added: "0.6V p-p"
- note added: "KU=3"
- note added: "KU=5.1"
- moved on the sheet: C?, R?, U?

Commit message: -  то, что успели нарисовать в свободное время
Parts:
- added C58: 100n, Capacitor_SMD:C_0603_1608Metric, symbol Device:C
- C26, C29: renamed from C?; footprint Capacitor_SMD:C_1206_3216Metric -> Capacitor_SMD:C_0603_1608Metric
- gave numbers to parts that had none: 75
Connections:
- net labels added: ADC12_INP5
- net labels removed: ADC12_INP4

Commit message: - вроде все провода соединили
Parts:
- added C59: 100n, Capacitor_SMD:C_0603_1608Metric, symbol Device:C
Connections:
- net +3.3VA: now also C59.1
- net GND: now also C59.2
Changed lines of the file:
@@
+	1    0    0    -1
+$EndComp
+$Comp
+L Device:C C59
+U 1 1 5DA77279
+P 1750 6350
+F 0 "C59" H 1865 6396 50  0000 L CNN
+F 1 "100n" H 1865 6305 50  0000 L CNN
+F 2 "Capacitor_SMD:C_0603_1608Metric" H 1788 6200 50  0001 C CNN
+F 3 "~" H 1750 6350 50  0001 C CNN
+	1    1750 6350
+	1    0    0    -1
+$EndComp
+$Comp
+L power:GND #PWR0191
+U 1 1 5DA77C49
+P 1750 6500
+F 0 "#PWR0191" H 1750 6250 50  0001 C CNN
+F 1 "GND" H 1755 6327 50  0001 C CNN
+F 2 "" H 1750 6500 50  0001 C CNN
+F 3 "" H 1750 6500 50  0001 C CNN
+	1    1750 6500
+	1    0    0    -1
+$EndComp
+$Comp
+L power:+3.3VA #PWR0192
+U 1 1 5DA7836E
+P 1750 6200
+F 0 "#PWR0192" H 1750 6050 50  0001 C CNN
+F 1 "+3.3VA" H 1765 6373 50  0000 C CNN
+F 2 "" H 1750 6200 50  0001 C CNN
+F 3 "" H 1750 6200 50  0001 C CNN
+	1    1750 6200
 	1    0    0    -1
 $EndComp

Commit message: - вынесли процессинг данных из прерывания
- начали отсылать данные на клиентскую часть, чтобы глянуть их
Parts:
- U13, U14: value AD8221BRMZ -> AD8221
Changed lines of the file:
@@
 P 7900 3350
 F 0 "U14" H 8150 3650 50  0000 L CNN
-F 1 "AD8221BRMZ" H 7950 3550 50  0000 L CNN
+F 1 "AD8221" H 7950 3550 50  0000 L CNN
 F 2 "Package_SO:MSOP-8_3x3mm_P0.65mm" H 7700 3350 50  0001 C CNN
 F 3 "https://www.analog.com/media/en/technical-documentation/data-sheets/AD8421.pdf" H 8250 2950 50  0001 C CNN
@@
 P 7750 5100
 F 0 "U13" H 8000 5400 50  0000 L CNN
-F 1 "AD8221BRMZ" H 7800 5300 50  0000 L CNN
+F 1 "AD8221" H 7800 5300 50  0000 L CNN
 F 2 "Package_SO:MSOP-8_3x3mm_P0.65mm" H 7550 5100 50  0001 C CNN
 F 3 "https://www.analog.com/media/en/technical-documentation/data-sheets/AD8421.pdf" H 8100 4700 50  0001 C CNN
