File: circuit/TestDSBGA6/TestDSBGA6.sch (KiCad schematic (older format))
At the start: 9 parts

Commit message: - залили тестовый проект, правда без папки Drivers ибо она слишком большая
Parts:
- gave numbers to parts that had none: 9
Changed lines of the file:
@@
 $EndDescr
 $Comp
-L Connector:USB_B_Micro J?
+L Connector:USB_B_Micro J1
 U 1 1 5DA8C49C
 P 2750 2750
-F 0 "J?" H 2807 3217 50  0000 C CNN
+F 0 "J1" H 2807 3217 50  0000 C CNN
 F 1 "USB_B_Micro" H 2807 3126 50  0000 C CNN
 F 2 "Connector_USB:USB_Micro-B_Molex-105017-0001" H 2900 2700 50  0001 C CNN
@@
 $EndComp
 $Comp
-L Device:LED D?
+L Device:LED D1
 U 1 1 5DA8CA21
 P 5350 3000
-F 0 "D?" V 5389 2883 50  0000 R CNN
+F 0 "D1" V 5389 2883 50  0000 R CNN
 F 1 "LED" V 5298 2883 50  0000 R CNN
 F 2 "LED_SMD:LED_0805_2012Metric_Pad1.15x1.40mm_HandSolder" H 5350 3000 50  0001 C CNN
@@
 $EndComp
 $Comp
-L Device:Battery_Cell BT?
+L Device:Battery_Cell BT1
 U 1 1 5DA8CDAD
 P 6000 3050
-F 0 "BT?" H 6118 3146 50  0000 L CNN
+F 0 "BT1" H 6118 3146 50  0000 L CNN
 F 1 "2.54mm" H 6118 3055 50  0000 L CNN
 F 2 "Connector_PinSocket_2.54mm:PinSocket_1x02_P2.54mm_Vertical" V 6000 3110 50  0001 C CNN
@@
 $EndComp
 $Comp
-L Device:Battery_Cell BT?
+L Device:Battery_Cell BT2
 U 1 1 5DA8D080
 P 6550 3050
-F 0 "BT?" H 6668 3146 50  0000 L CNN
+F 0 "BT2" H 6668 3146 50  0000 L CNN
 F 1 "1.25mm" H 6668 3055 50  0000 L CNN
 F 2 "Connector_PinSocket_1.27mm:PinSocket_1x02_P1.27mm_Vertical" V 6550 3110 50  0001 C CNN
@@
 $EndComp
 $Comp
-L balmer:BQ25101 U?
+L balmer:BQ25101 U1
 U 1 1 5DA8E8E9
 P 4450 2800
-F 0 "U?" H 4425 3175 50  0000 C CNN
+F 0 "U1" H 4425 3175 50  0000 C CNN
 F 1 "BQ25101" H 4425 3084 50  0000 C CNN
 F 2 "balmer:DSBGA-6_0.4mm" H 4500 2800 50  0001 C CNN
@@
 $EndComp
 $Comp
-L Device:C C?
+L Device:C C1
 U 1 1 5DA8F887
 P 3350 3150
-F 0 "C?" H 3465 3196 50  0000 L CNN
+F 0 "C1" H 3465 3196 50  0000 L CNN
 F 1 "1u" H 3465 3105 50  0000 L CNN
 F 2 "Capacitor_SMD:C_0805_2012Metric" H 3388 3000 50  0001 C CNN
@@
 $EndComp
 $Comp
-L Device:R R?
+L Device:R R2
 U 1 1 5DA8FE0A
 P 3650 3150
-F 0 "R?" H 3720 3196 50  0000 L CNN
+F 0 "R2" H 3720 3196 50  0000 L CNN
 F 1 "10k" H 3720 3105 50  0000 L CNN
 F 2 "Resistor_SMD:R_0603_1608Metric" V 3580 3150 50  0001 C CNN
@@
 $EndComp
 $Comp
-L Device:R R?
+L Device:R R3
 U 1 1 5DA903B5
 P 3950 3150
-F 0 "R?" H 4020 3196 50  0000 L CNN
+F 0 "R3" H 4020 3196 50  0000 L CNN
 F 1 "3.3k" H 4020 3105 50  0000 L CNN
 F 2 "Resistor_SMD:R_0603_1608Metric" V 3880 3150 50  0001 C CNN
@@
 $EndComp
 $Comp
-L Device:R R?
+L Device:R R1
 U 1 1 5DA91ADB
 P 4950 3000
-F 0 "R?" H 5020 3046 50  0000 L CNN
+F 0 "R1" H 5020 3046 50  0000 L CNN
 F 1 "1k" H 5020 2955 50  0000 L CNN
 F 2 "Resistor_SMD:R_0603_1608Metric" V 4880 3000 50  0001 C CNN
@@
 $EndComp
 $Comp
-L power:GND #PWR?
+L power:GND #PWR0101
 U 1 1 5DA93B7A
 P 4450 3350
-F 0 "#PWR?" H 4450 3100 50  0001 C CNN
+F 0 "#PWR0101" H 4450 3100 50  0001 C CNN
 F 1 "GND" H 4455 3177 50  0001 C CNN
 F 2 "" H 4450 3350 50  0001 C CNN
