File: circuit/RLCMeterH750_v2/RLCMeterH750_v2.kicad_pcb (KiCad board)
At the start: 2 copper layers, 80 x 65 mm, 163 parts, among them J1 SWD, J2 USB_B_Micro, J3 ILI_9321(2.2inch), J4 DUT, SW1 EVQWKL001, SW2 PowerOn, U1 STM32H750VITx, U10 AD8031, U11 AD8031, U12 AD9833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

Commit message: - не до конца разведенная вторая версия платы
Parts:
- removed C20, C23: 100n, Capacitor_SMD:C_0603_1608Metric
- removed C62: 220u, Capacitor_SMD:CP_Elec_6.3x5.7
- C61: value 220u -> 100u; footprint Capacitor_SMD:CP_Elec_6.3x5.7 -> Capacitor_SMD:C_1206_3216Metric
- moved C63 75.2 mm to (150.2, 138.3)
- moved C64 51.6 mm to (143.7, 119.3)
- moved L4 50.6 mm to (142.8, 109.5), turned to 270 degrees
- moved L3 47.8 mm to (145.8, 109.5), turned to 270 degrees
- moved U18 38.3 mm to (152.8, 106.7), turned to 90 degrees
- moved C60 35.4 mm to (144.3, 93.9), turned to 90 degrees
- moved C24 30.3 mm to (135.5, 96.6), turned to 90 degrees
- moved L2 29.6 mm to (146.5, 98.0), turned to 180 degrees
- moved C61 19.8 mm to (155.2, 110.8), turned to 180 degrees
- moved C21 17.8 mm to (149.8, 124.9)
- moved U6 11.7 mm to (139.6, 93.7)
- moved C14 10.9 mm to (118.1, 96.7)
- moved R22 10.4 mm to (146.7, 94.7), turned to 270 degrees
- moved C18 9.27 mm to (110.3, 99.5), turned to 180 degrees
- moved C15 6.59 mm to (111.1, 93.3)
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Routing:
- net +5V: track 109.4 -> 47.5 mm, vias 9 -> 6
- net +3.3VA: track 49.6 -> 102.0 mm, vias 8 -> 12
- net Net-(C15-Pad1): track 0.00 -> 49.8 mm, vias 0 -> 1
- net +3V3: track 179.7 -> 142.7 mm, vias 2 -> 1
- net +BATT: track 37.0 -> 69.3 mm
- net Net-(C16-Pad1): track 0.00 -> 27.2 mm, vias 0 -> 3
- net Net-(C66-Pad1): track 1.96 -> 16.8 mm, vias 0 -> 2
- net -2V5: track 123.6 -> 111.4 mm, vias 6 -> 5
- net Net-(C67-Pad1): track 2.01 -> 13.4 mm, vias 0 -> 2
- net Net-(C60-Pad1): track 0.00 -> 9.34 mm
- net Net-(C21-Pad1): track 0.00 -> 4.85 mm
- net Net-(C12-Pad2): track 0.00 -> 3.87 mm
- net Net-(C14-Pad2): track 0.00 -> 2.61 mm
- net Net-(C12-Pad1): track 0.00 -> 2.45 mm
- net GND: track 211.6 -> 213.8 mm, vias 173 -> 167
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Other:
- board text added: "BalmerDX 2020"
- board text removed: "BalmerDX 2019"

Commit message: - все дорожки развели
Parts:
- added C20: 100n, Capacitor_SMD:C_0603_1608Metric, F.Cu at (110.5, 108.5)
- moved C46 0.14 mm to (149.4, 136.4)
- moved R45 0.06 mm to (137.9, 124.6)
Connections:
- SW1 pad GND: (no net) -> GND
- SW1 pad PAD: (no net) -> GND
Routing:
- net +5V: track 47.5 -> 113.5 mm, vias 6 -> 8
- net +3.3VA: track 102.0 -> 148.3 mm, vias 12 -> 15
- net GND: track 213.8 -> 230.5 mm, vias 167 -> 171
- net -2V5: track 111.4 -> 114.8 mm, vias 5 -> 7
