File: circuit/RLCMeterH750_v2/RLCMeterH750_v2.kicad_pcb (KiCad board)
At the start: 2 copper layers, 80 x 65 mm, 161 parts, among them J1 SWD, J2 USB_B_Micro, J3 ILI_9321(2.2inch), J4 DUT, SW1 EVQWKL001, SW2 PowerOn, U1 STM32H750VITx, U10 AD8031, U11 AD8031, U12 AD9833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

Commit message: - более узкий корпус для m25p16
Parts:
- U7: footprint Package_SO:SOIC-8_5.23x5.23mm_P1.27mm -> Package_SO:SOIC-8_3.9x4.9mm_P1.27mm
Routing:
- net /FLASH_MISO: track 6.69 -> 9.49 mm
- net /ENC_B: track 23.0 -> 24.5 mm
- net /FLASH_CS: track 3.89 -> 5.07 mm
- net +3V3: track 142.7 -> 143.4 mm
- net /FLASH_SCK: track 11.3 -> 11.9 mm
