File: circuit/RLCMeterH750_v2/RLCMeterH750_v2.sch (KiCad schematic (older format))
At the start: 68 parts, among them J1 SWD, J2 USB_B_Micro, J3 ILI_9321(2.2inch), SW1 EVQWKL001, SW2 PowerOn, U1 STM32H750VITx, U18 HT7333, U2 ISL9204, U3 LTC1550LCS8-2, U4 TPS60241DGKR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

Commit message: - не до конца разведенная вторая версия платы
Parts:
- removed C20, C23: 100n, Capacitor_SMD:C_0603_1608Metric, symbol Device:C
- removed C61, C62: 220u, Capacitor_SMD:CP_Elec_6.3x5.7, symbol Device:CP
- added C61: 100u, Capacitor_SMD:C_1206_3216Metric, symbol Device:C
Connections:
- wire segments 242 -> 237
Changed lines of the file:
@@
 EESchema Schematic File Version 4
-LIBS:RLCMeterH750_v2-cache
 EELAYER 30 0
 EELAYER END
@@
 	1    0    0    -1
 $EndComp
-$Comp
-L Device:C C20
-U 1 1 5DA0BEF5
-P 7250 5900
-F 0 "C20" H 7365 5946 50  0000 L CNN
-F 1 "100n" H 7365 5855 50  0000 L CNN
-F 2 "Capacitor_SMD:C_0603_1608Metric" H 7288 5750 50  0001 C CNN
-F 3 "~" H 7250 5900 50  0001 C CNN
-	1    7250 5900
-	1    0    0    -1
-$EndComp
-Wire Wire Line
-	7700 6050 7250 6050
-Connection ~ 7250 6050
-Wire Wire Line
-	7700 5750 7250 5750
-Connection ~ 7250 5750
 Wire Wire Line
 	7250 5700 7250 5750
@@
 Wire Wire Line
 	9400 2500 9400 2550
-$Comp
-L Device:C C23
-U 1 1 5DA2CFDE
-P 10600 1950
-F 0 "C23" H 10715 1996 50  0000 L CNN
-F 1 "100n" H 10715 1905 50  0000 L CNN
-F 2 "Capacitor_SMD:C_0603_1608Metric" H 10638 1800 50  0001 C CNN
-F 3 "~" H 10600 1950 50  0001 C CNN
-	1    10600 1950
-	1    0    0    -1
-$EndComp
 Wire Wire Line
 	10300 2200 10350 2200
@@
 	10350 1800 10350 2200
 Connection ~ 10350 1800
-$Comp
-L power:GND #PWR0141
-U 1 1 5DA4448D
-P 10600 2100
-F 0 "#PWR0141" H 10600 1850 50  0001 C CNN
-F 1 "GND" H 10605 1927 50  0001 C CNN
-F 2 "" H 10600 2100 50  0001 C CNN
-F 3 "" H 10600 2100 50  0001 C CNN
-	1    10600 2100
-	1    0    0    -1
-$EndComp
-Wire Wire Line
-	10350 1800 10600 1800
 Wire Wire Line
 	10300 2400 10650 2400
@@
 	4650 1750 4750 1750
 $Comp
-L Device:CP C61
-U 1 1 5DE6DB52
-P 7700 5900
-F 0 "C61" H 7818 5946 50  0000 L CNN
-F 1 "220u" H 7818 5855 50  0000 L CNN
-F 2 "Capacitor_SMD:CP_Elec_6.3x5.7" H 7738 5750 50  0001 C CNN
-F 3 "~" H 7700 5900 50  0001 C CNN
-	1    7700 5900
-	1    0    0    -1
-$EndComp
-$Comp
-L Device:CP C62
-U 1 1 5DE7058A
-P 8150 5900
-F 0 "C62" H 8268 5946 50  0000 L CNN
-F 1 "220u" H 8268 5855 50  0000 L CNN
-F 2 "Capacitor_SMD:CP_Elec_6.3x5.7" H 8188 5750 50  0001 C CNN
-F 3 "~" H 8150 5900 50  0001 C CNN
-	1    8150 5900
-	1    0    0    -1
-$EndComp
-Wire Wire Line
-	7700 6050 8150 6050
-Connection ~ 7700 6050
-Wire Wire Line
-	7700 5750 8150 5750
-Connection ~ 7700 5750
+L Device:C C61
+U 1 1 5DE60A32
+P 7250 5900
+F 0 "C61" H 7365 5946 50  0000 L CNN
+F 1 "100u" H 7365 5855 50  0000 L CNN
+F 2 "Capacitor_SMD:C_1206_3216Metric" H 7288 5750 50  0001 C CNN
+F 3 "~" H 7250 5900 50  0001 C CNN
+	1    7250 5900
+	1    0    0    -1
+$EndComp
 $EndSCHEMATC

Commit message: - более узкий корпус для m25p16
Parts:
- U7: footprint Package_SO:SOIC-8_5.23x5.23mm_P1.27mm -> Package_SO:SOIC-8_3.9x4.9mm_P1.27mm
Changed lines of the file:
@@
 F 0 "U7" H 9875 2747 60  0000 C CNN
 F 1 "M25P16" H 9875 2641 60  0000 C CNN
-F 2 "Package_SO:SOIC-8_5.23x5.23mm_P1.27mm" H 9900 2350 60  0001 C CNN
+F 2 "Package_SO:SOIC-8_3.9x4.9mm_P1.27mm" H 9900 2350 60  0001 C CNN
 F 3 "" H 9900 2350 60  0001 C CNN
 	1    9850 2350
