File: circuit/RLCMeterH750_v2/analog.sch (KiCad schematic (older format))
At the start: 91 parts, among them J4 DUT, U10 AD8031, U11 AD8031, U12 AD9833, U13 AD8221, U14 AD8221, U15 AD8031, U16 AD8031, U17 AD8031, U19 FSA3357L8X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

Commit message: - все дорожки развели
Parts:
- added C20: 100n, Capacitor_SMD:C_0603_1608Metric, symbol Device:C
Connections:
- net +5V: now also C20.1
- net GND: now also C20.2
Changed lines of the file:
@@
 Text GLabel 7200 350  0    50   Input ~ 0
 KU_V
+$Comp
+L Device:C C20
+U 1 1 5DEC9EFE
+P 4350 1150
+F 0 "C20" H 4465 1196 50  0000 L CNN
+F 1 "100n" H 4465 1105 50  0000 L CNN
+F 2 "Capacitor_SMD:C_0603_1608Metric" H 4388 1000 50  0001 C CNN
+F 3 "~" H 4350 1150 50  0001 C CNN
+	1    4350 1150
+	1    0    0    -1
+$EndComp
+$Comp
+L power:GND #PWR0141
+U 1 1 5DECA129
+P 4350 1300
+F 0 "#PWR0141" H 4350 1050 50  0001 C CNN
+F 1 "GND" H 4355 1127 50  0001 C CNN
+F 2 "" H 4350 1300 50  0001 C CNN
+F 3 "" H 4350 1300 50  0001 C CNN
+	1    4350 1300
+	1    0    0    -1
+$EndComp
+$Comp
+L power:+5V #PWR0206
+U 1 1 5DECA2AF
+P 4350 1000
+F 0 "#PWR0206" H 4350 850 50  0001 C CNN
+F 1 "+5V" H 4365 1173 50  0000 C CNN
+F 2 "" H 4350 1000 50  0001 C CNN
+F 3 "" H 4350 1000 50  0001 C CNN
+	1    4350 1000
+	1    0    0    -1
+$EndComp
 $EndSCHEMATC

Commit message: - исправили схему для большей точности на 400 Гц (криво правда, потом еще поправим)
- plot теперь корректно очищает линию на краях интервала
- scene_graph можно возюкать линией туда-сюда
Parts:
- added C?: 470u, symbol Device:CP
Connections:
- net +1V5: now also C?.1
- net GND: now also C?.2
Other:
- note added: "Без этого конденсатора\nчастота резонанса 400 Гц\n470 uF изменяет частоту\nрезонанса до 140 Гц\n2200 uF изменяет частоту\nрезонанса до 65 Гц"
Changed lines of the file:
@@
 	1    0    0    -1
 $EndComp
+$Comp
+L Device:CP C?
+U 1 1 5E098957
+P 2950 1500
+F 0 "C?" H 3068 1546 50  0000 L CNN
+F 1 "470u" H 3068 1455 50  0000 L CNN
+F 2 "" H 2988 1350 50  0001 C CNN
+F 3 "~" H 2950 1500 50  0001 C CNN
+	1    2950 1500
+	1    0    0    -1
+$EndComp
+Wire Wire Line
+	2950 1650 2450 1650
+Connection ~ 2450 1650
+Wire Wire Line
+	2450 1250 2950 1250
+Wire Wire Line
+	2950 1250 2950 1350
+Connection ~ 2450 1250
+Text Notes 2650 1200 0    50   ~ 0
+Без этого конденсатора\nчастота резонанса 400 Гц\n470 uF изменяет частоту\nрезонанса до 140 Гц\n2200 uF изменяет частоту\nрезонанса до 65 Гц
 $EndSCHEMATC
